File: pcb/main-keyboard/keyboard/keyboard.kicad_sch (KiCad schematic)
At the start: 132 parts

Commit message: Update specs to match actual design changes: RP2040 Plus module, monochrome OLED, magnetic connector, PCF8574 expander, 14x5 matrix
Parts:
- added A1: RaspberryPi_Pico_W, Module:RaspberryPi_Pico_W_SMD_HandSolder, symbol MCU_Module:RaspberryPi_Pico_W
- added F1, F2: Fuse, symbol Device:Fuse
- added J1: Conn_01x06_Pin, symbol Connector:Conn_01x06_Pin
- added J2: Conn_01x02_Pin, Connector_JST:JST_ZE_S02B-ZESK-2D_1x02_P1.50mm_Horizontal, symbol Connector:Conn_01x02_Pin
- added J3: Conn_01x06_Socket, Connector:Tag-Connect_TC2030-IDC-NL_2x03_P1.27mm_Vertical, symbol Connector:Conn_01x06_Socket
- added P1: USB_C_Plug_USB2.0, symbol Connector:USB_C_Plug_USB2.0
- added R2: R, symbol Device:R
- added R3, R4: R, Custom Footprints:R_0402_Clean, symbol Device:R
- added U2: NRF24L01_Breakout, RF_Module:nRF24L01_Breakout, symbol RF:NRF24L01_Breakout
- added U3: TP4056-42-ESOP8, Package_SO:SOIC-8-1EP_3.9x4.9mm_P1.27mm_EP2.41x3.3mm, symbol Battery_Management:TP4056-42-ESOP8
- added U5: SSD1327-OLED, Custom Footprints:SSD1327-128x128-OLED, symbol Custom Library:SSD1327-OLED
- added Y1: Crystal, symbol Device:Crystal
Connections:
- new net: P1.A6 (D+), R2.1
- new net: J2.1 (Pin_1), U3.5 (BAT)
- new net: A1.13 (GND), A1.18 (GND), A1.23 (GND), A1.28 (GND), A1.3 (GND), A1.38 (GND), A1.8 (GND), J2.2 (Pin_2), U2.1 (GND), U3.3 (GND)
- new net: A1.36 (3V3), U2.2 (VCC), U5.2 (Vcc)
- new net: A1.20 (GPIO15), U2.3 (CE)
- new net: A1.21 (GPIO16), U2.4 (~{CSN})
- new net: A1.26 (GPIO20), U2.5 (SCK)
- new net: A1.24 (GPIO18), U2.6 (MOSI)
- new net: A1.25 (GPIO19), U2.7 (MISO)
- new net: A1.22 (GPIO17), U2.8 (IRQ)
- new net: P1.A1 (GND), P1.A12 (GND), P1.B1 (GND), P1.B12 (GND)
- new net: P1.A4 (VBUS), P1.A9 (VBUS), P1.B4 (VBUS), P1.B9 (VBUS)
- new net: P1.A7 (D-), R3.1
- new net: A1.40 (VBUS), F2.2
- new net: F2.1, U3.4 (V_{CC})
Other:
- moved on the sheet: D1, D10, D11, D12, D13, D15, D16, D17, D18, D19, D2, D20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
